File: hardware/Homegreen Node Basic/user_interface.kicad_sch (KiCad schematic)
At the start: 21 parts, among them U2 TM1637, U3 FJ3661BH, U4 TTP224

Commit message: Kicad update
Parts:
- renumbered C2 to C10, C2 to C11, C2 to C12, C2 to C13, C2 to C8, C2 to C9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
